Commit message: feat: 相机改为外置支架安装（eye-to-hand），URDF 补齐末端与相机坐标系
方案变更：相机不再装在机械臂末端，而是额外架一个深度相机俯视工作台。

这是一个实质性简化，消掉了原先两个最麻烦的问题：
- 标定只做一次，不再被碰撞、更换夹爪破坏（原先会静默失效，症状是
  「抓取随机失败」，极难定位）
- 没有手指盲区，抓取全程可见

代价是需要新增两条风险，都已写入方案文档：
- R12 机械臂本体可能遮挡外置相机视线。装支架之前必须先手动走一遍
  工作范围，从相机位置确认视线不被挡——这是外置相机最容易被忽略的坑
- R13 相机距离远，像素误差折算成实际位移更大

URDF（阶段 1 前半）：
- 新增 world 根节点与 world_to_base 虚拟关节，MoveIt 需要
- 新增 tool0（末端法兰）、gripper_tcp（抓取参考点，MoveIt 规划链终点）
- 新增 camera_link，挂在 base_link 下（外置固定相机）
- 新增 camera_color_optical_frame，含 REP-103 到光学坐标系的标准变换
- 相机安装参数提取为 xacro 属性，便于手眼标定后替换

文档同步更新：架构图、坐标链接说明、阶段 6 流程、风险表 R4/R8，
以及手眼标定章节改写为 eye-to-hand（标的是 base_link 到 camera_link，
标定板固定在末端随臂运动）。

新增工具：
- tools/check_urdf.py        离线校验 URDF 结构：XML 合法性、父子引用、
                             树连通性、xacro 属性引用、必需坐标系
- tools/fix_line_endings.ps1 CRLF 批量转 LF，字节级操作

关于换行符：上游代码库本身是 CRLF（156 个文件）。git 索引与 blob 中
一直是 LF（已用 git cat-file 逐字节验证），所以推到 GitHub 的内容是
干净的，虚拟机上 clone 出来也是 LF。本次把 Windows 工作区也统一为 LF，
避免 xacro 等文件在 Ubuntu 上出错。

注意 tools/fix_line_endings.ps1 刻意不解析 git ls-files 的输出：
PowerShell 5.1 收到的是带八进制转义的路径，本仓库 docs/ 下有中文文件名，
直接用会报「路径中具有非法字符」。改为从文件系统枚举。

验证：URDF 检查 0 问题（15 links / 14 joints / 根节点 world / 全部连通）；
Python 语法 132 文件 0 失败；全仓库无 CRLF 残留。

File: dummy_vc_ws/src/dummy2_urdf/urdf/dummy2_urdf.xacro (robot description, xacro)
@@ -4,4 +4,30 @@
 <xacro:include filename="$(find dummy2_urdf_description)/urdf/dummy2_urdf.trans" />
 <xacro:include filename="$(find dummy2_urdf_description)/urdf/dummy2_urdf.gazebo" />
+<!-- ==========================================================================
+     可调参数
+     ==========================================================================
+     下面这几个值决定夹持点和相机在模型里的位置。凡是标了「实测」的，
+     都要按 docs/02-阶段0标定操作手册.md 量出来再改。
+     数值偏 5 mm，IK 就会把末端整体偏移 5 mm，抓取时表现为
+     「对准了但没夹住」——而且你会先怀疑视觉，浪费大量时间在后处理上。
+     ========================================================================== -->
+<!-- 手指伸出的方向：URDF 里手爪挂在 link7 的 +y 方向 -->
+<xacro:property name="hand_axis" value="y"/>
+<!-- link7 -> 两指夹持中心(指尖前端中点)，沿 hand_axis 的距离。实测 -->
+<xacro:property name="tcp_offset_y" value="0.06"/>
+<!-- 相机的安装参数（外置支架，eye-to-hand）定义在文件末尾的相机段落里，
+     因为那里有较长的说明。用 grep 搜 camera_offset 可以找到。 -->
+<!-- ==========================================================================
+     基座虚拟关节
+     ==========================================================================
+     MoveIt 需要一个能把机械臂固定到某个世界坐标系的虚拟关节。
+     固定式（而非浮动式）意味着机械臂底座在规划中不可移动。
+     ========================================================================== -->
+<link name="world"/>
+<joint name="world_to_base" type="fixed">
+  <origin xyz="0 0 0" rpy="0 0 0"/>
+  <parent link="world"/>
+  <child link="base_link"/>
+</joint>
 <link name="base_link">
   <inertial>
@@ -265,3 +291,71 @@
   <limit upper="0.023" lower="0.0" effort="100" velocity="100"/>
 </joint>
+<!-- ==========================================================================
+     末端坐标系（阶段 1 新增）
+     ==========================================================================
+     原来的 URDF 到 dummy_hand_v1_1 就结束了，没有 TCP、没有相机坐标系，
+     所以无法定义 MoveIt 的规划链，也无法把图像投到基座坐标系。
+     坐标链（注意：XML 注释里不能出现连续两个连字符，所以这里用箭头文字替代）
+       link7_v1_1  ->  tool0  ->  gripper_tcp
+                           ->  camera_link  ->  camera_color_optical_frame
+     ========================================================================== -->
+<!-- tool0：末端法兰坐标，与手爪根部重合，便于标定和参考项目对齐 -->
+<link name="tool0"/>
+<joint name="tool0_joint" type="fixed">
+  <origin xyz="0 0.052312 0" rpy="0 0 0"/>
+  <parent link="link7_v1_1"/>
+  <child link="tool0"/>
+</joint>
+<!-- gripper_tcp：抓取参考点。MoveIt 的规划链终点用这个，不用 link7。
+     偏移量必须实测：从手爪根部到两指指尖前端的中点。 -->
+<link name="gripper_tcp"/>
+<joint name="gripper_tcp_joint" type="fixed">
+  <origin xyz="0 ${tcp_offset_y - 0.052312} 0" rpy="0 0 0"/>
+  <parent link="tool0"/>
+  <child link="gripper_tcp"/>
+</joint>
+<!-- camera_link：相机本体坐标系（x 前、y 左、z 上，符合 REP-103）
+     相机是**外置支架固定安装**（eye-to-hand），所以这个坐标系挂在 base_link
+     下，而不是末端。这样标定只需要做一次，且不会被碰撞或更换夹爪破坏，
+     抓取过程中相机也不会被手指遮挡。
+     MASTER 与 FALLBACK 的关系：
+       标定完成后，base_link 到 camera_link 的变换由外部静态 TF 发布
+       （见下方说明），本文件里这个固定关节只作为**没有标定时的兜底**，
+       让你在 RViz 里至少能看到相机坐标系。
+       两个变换同时存在会让 TF 树出现两个 base_link 到 camera_link 的发布者，
+       tf2 会报 "TF_MULTIPLE_AUTHORITIES"。所以标定完成后必须二选一：
+         方案 A（推荐）：把标定结果填进下面这个固定关节，删掉外部静态发布
+         方案 B：给下面这个关节加条件，标定后不再展开
+       首期用方案 A，简单直接。 -->
+<xacro:property name="camera_offset_x" value="0.30"/>
+<xacro:property name="camera_offset_y" value="0.0"/>
+<xacro:property name="camera_offset_z" value="0.60"/>
+<!-- 相机安装姿态（度）。外置俯视支架通常是「朝下看」，
+     对应绕 x 轴 -90°；然后再绕 z 轴转一个安装偏航角。
+     这些都是标定前的估计值，手眼标定会给出准确结果。 -->
+<xacro:property name="camera_mount_roll_deg" value="180"/>
+<xacro:property name="camera_mount_pitch_deg" value="0"/>
+<xacro:property name="camera_mount_yaw_deg" value="0"/>
+<link name="camera_link"/>
+<joint name="camera_link_joint" type="fixed">
+  <origin xyz="${camera_offset_x} ${camera_offset_y} ${camera_offset_z}"
+          rpy="${camera_mount_roll_deg * pi / 180} ${camera_mount_pitch_deg * pi / 180} ${camera_mount_yaw_deg * pi / 180}"/>
+  <parent link="base_link"/>
+  <child link="camera_link"/>
+</joint>
+<!-- camera_color_optical_frame：光学坐标系（z 前、x 右、y 下）。
+     注意 optical frame 的轴向约定与 REP-103 不同，这是写视觉变换时最容易
+     翻车的地方：图像的 x 对应光学系的 x（右），图像的 y 对应光学系的 y（下），
+     深度对应光学系的 z（前，正值朝景物）。
+     RealSense 的 realsense2_camera 节点会自己发布 camera_link 到
+     camera_color_optical_frame，所以接了真实驱动后这里会被覆盖；
+     保留它是为了没有相机时 RViz 里也能看到坐标系。
+     rpy="-1.5707963 0 -1.5707963" 是 REP-103 -> 光学系的标准变换：
+     绕 x 转 -90° 把 z 从朝上掰到朝前，再绕 z 转 -90° 对齐 x/y。 -->
+<link name="camera_color_optical_frame"/>
+<joint name="camera_optical_joint" type="fixed">
+  <origin xyz="0 0 0" rpy="-1.5707963 0 -1.5707963"/>
+  <parent link="camera_link"/>
+  <child link="camera_color_optical_frame"/>
+</joint>
 </robot>

Commit message: ﻿feat: 关节限位改为设备实测行程；新增 check_urdf_limits 守住这个不变量
## 背景：阶段 1 已完成，下一步是阶段 2（MoveIt）

核对 URDF 发现阶段 1 的要求全部满足了：`world` link + `world_to_base` 虚拟
关节、`tool0`、`gripper_tcp`、`camera_link`、`camera_color_optical_frame`
都在。所以 MoveIt 的输入已经齐了。

但**关节限位是错的**，而这是 MoveIt 之前必须先修的。

## 问题

设备会**静默丢弃**含有它不接受的 move_j 值的整条命令。所以 **URDF 限位比设备
宽不是"无害的取整差异"** —— MoveIt 会规划进那段范围，驱动忠实地换算，然后
设备把整条命令丢掉，日志里什么都没有。这正是 j3 长时间看起来像"死关节"的
同一个机制。

把 URDF 限位换算到设备可接受区间后对比：

    joint     旧 URDF 限位      设备可接受        问题
    joint_1   ±180           ±165            两侧各宽 15 度
    joint_2   -120..+75      -90..+75        下限宽 30 度
    joint_3    -90..+75      -90..+45        上限宽 30 度
    joint_4   ±180           -180..+165      上限宽 15 度（腕关节，转得最快）
    joint_5   ±100           -90..+90        两侧各宽 10 度
    joint_6   ±180           ±180            一致

换算关系：`urdf_deg = sign * (move_j - movej_urdf_zero_deg)`。

## 修改

六个限位全部改为**设备实测行程**，取整方向朝外（下限 floor、上限 ceil），
保证不会比实测区间更紧：

    joint_1  ±165          joint_4  -180..+165
    joint_2  -90..+75      joint_5  -90..+90
    joint_3  -90..+45      joint_6  ±180

两个命名姿态仍可到达：

    home   urdf [0, 0, 0, 0, 0, 0]
    reset  urdf [0, +75, -90, 0, 0, 0]     ← j2/j3 正好落在限位上

**j3 下限保持 -90 不能动**：断电收缩姿态正好就是 -90，没有余量可让。
j3 上限从 +75 收到 +45，这是本次最要紧的一处。

xacro 里写了一段说明，解释这些值来自实测而不是厂商数据，以及为什么"限位比
设备宽"是危险的。

## 新增回归检查 check_urdf_limits.py

限位在两个文件里（xacro 的弧度、yaml 的 movej_accepted_range_deg），本次是
把两边对齐。这个脚本守住这个不变量：把两侧都换算成 URDF 度，要求 **URDF 限位
不超出设备可接受范围**（容差 1 度，因为限位是实测值朝外取整来的），并且两个
命名姿态仍在限位内。

已加入 run_checks.py，现在共 10 项离线检查全过。

## 顺带修好 run_checks.py

上一轮我改到一半留下一个跑不起来的文件：CHECKS 元组加了第四个元素但循环还在
按三个解包，且 check_encoding.py 需要显式文件列表（不带参数只打印用法）。
两处都修了；输出还加了编码保护（Windows 控制台常是 GBK，子进程输出里的
U+FFFD 会让 print 抛异常，把报告本身吞掉）。

验证：语法 160 文件 0 失败；check_urdf 通过；10 项离线检查全过；
编码 3 文件无问题；无 CRLF 残留。

File: dummy_vc_ws/src/dummy2_urdf/urdf/dummy2_urdf.xacro (robot description, xacro)
@@ -235,5 +235,24 @@
   <child link="link1_v1_1"/>
   <axis xyz="0.0 -0.0 -1.0"/>
-  <limit upper="3.141593" lower="-3.141593" effort="100" velocity="100"/>
+  <!--
+    Limits throughout this file are the DEVICE's real travel, measured with
+    tools/probe_range.py and classified with tools/analyse_range.py. They are
+    NOT the vendor's datasheet values, and the difference matters: the device
+    silently drops an entire command that contains a move_j value it will not
+    act on, so a limit that is looser than the device lets MoveIt plan a motion
+    the arm will then ignore with no error anywhere.
+    Mapping used for every joint:
+        urdf_deg = sign * (move_j - movej_urdf_zero_deg)
+    with sign = [-1, -1, -1, 1, -1, -1] and
+    movej_urdf_zero_deg = [0, 0, 90, 0, 0, 0].
+    Accepted move_j per joint, measured:
+        joint_1 [-165, 165]     joint_4 [-180, 165]
+        joint_2 [ -75,  90]     joint_5 [ -90,  90]
+        joint_3 [  45, 180]     joint_6 [-180, 180]
+    Bounds here are rounded outward from the measurements (floor for the lower,
+    ceil for the upper) so they are never tighter than what was observed.
+    tools/check_urdf_limits.py enforces that they are at least not looser.
+  -->
+  <limit upper="2.879793" lower="-2.879793" effort="100" velocity="100"/>
 </joint>
 <joint name="dummy2_joint2" type="revolute">
@@ -242,5 +261,20 @@
   <child link="link2_3_v4_1"/>
   <axis xyz="1.0 0.0 0.0"/>
-  <limit upper="1.308997" lower="-2.094395" effort="100" velocity="100"/>
+  <!--
+    Limits below are the DEVICE's real travel, not the vendor's datasheet, and
+    they come from measuring what move_j the arm will actually accept
+    (tools/probe_range.py, classified with tools/analyse_range.py).
+    The device silently drops a command containing a value it will not act on,
+    taking the whole command with it. So a limit here that is LOOSER than the
+    device is not a harmless rounding difference; MoveIt will happily plan
+    into it and the arm will simply not move.
+    Mapping used: urdf_deg = sign * (move_j - movej_urdf_zero_deg), with
+    sign = -1 and movej_urdf_zero_deg = 0 for joint_2, so
+        move_j [-75, 90]  ->  urdf [-90, 75].   upper matches exactly;
+        the lower bound here was -120, which the device cannot reach.
+    The retracted (power-off) pose is urdf joint_2 = +75, which rests exactly on
+    this upper limit.
+  -->
+  <limit upper="1.308997" lower="-1.570796" effort="100" velocity="100"/>
 </joint>
 <joint name="dummy2_joint3" type="revolute">
@@ -249,5 +283,16 @@
   <child link="link4_v3_1"/>
   <axis xyz="1.0 -0.0 0.0"/>
-  <limit upper="1.308997" lower="-1.570796" effort="100" velocity="100"/>
+  <!--
+    Device travel, measured. move_j [45, 180] with sign = -1 and
+    movej_urdf_zero_deg = 90 gives
+        urdf = -(move_j - 90)   ->   move_j 45  ->  urdf +45
+                                     move_j 180 ->  urdf -90
+    so urdf is [-90, +45]. The upper bound here was 1.308997 (+75), which is
+    30 deg past anything the device will accept: MoveIt could plan joint_3 to
+    +60 and the arm would ignore the entire command. Tightened to +45.
+    The lower bound stays at -90 because the retracted (power-off) pose is
+    exactly urdf joint_3 = -90, so there is no margin to give away.
+  -->
+  <limit upper="0.785398" lower="-1.570796" effort="100" velocity="100"/>
 </joint>
 <joint name="dummy2_joint4" type="revolute">
@@ -256,5 +301,5 @@
   <child link="link5_v3_1"/>
   <axis xyz="-0.0 1.0 0.0"/>
-  <limit upper="3.141593" lower="-3.141593" effort="100" velocity="100"/>
+  <limit upper="2.879793" lower="-3.141593" effort="100" velocity="100"/>
 </joint>
 <joint name="dummy2_joint5" type="revolute">
@@ -263,5 +308,5 @@
   <child link="link6_v3_1"/>
   <axis xyz="1.0 0.0 0.0"/>
-  <limit upper="1.745329" lower="-1.745329" effort="100" velocity="100"/>
+  <limit upper="1.570796" lower="-1.570796" effort="100" velocity="100"/>
 </joint>
 <joint name="dummy2_joint6" type="revolute">

Commit message: feat: 把实测的三个数写进模型 —— 无桌面、TCP 15 mm、24 mm 方块
用户给了三个数，替换掉之前全是 placeholder 的占位值：没有桌子（工件和
底座同一平面，所以工作面 z = 0）、link7 端面到两指夹持中心约 15 mm、
方块边长 24 mm。

为什么 TCP 从 0.06 改成 0.015 值得单独说：它比 hand 关节的 0.052312 还小，
于是 gripper_tcp 落到 hand 坐标系原点后方 y = -0.037312。这说明 URDF 里
那套手指几何（原作者模型）与实物不符：做碰撞感知规划前必须换成简化碰撞体，
否则会拿着 52 mm 长的假手掌去判断碰撞；并且 TCP 内移 45 mm，实际可达范围
比按原模型算的窄。同一个数写在两处（xacro 给 MoveIt 用，geometry.py 给
抓取点用），所以自测里加了一条交叉检查 —— 改一处忘另一处，规划和视觉就会
差几毫米，而那正好是"对准了却没夹住"的样子。

顺带：
- geometry.project_scene_measurements() 是本机的实测值，
  default_scene_measurements() 故意保持全占位，好让占位那条路径一直被测到
- 自测加第 9b 组：本机三个数都必须标 measured、必须与 xacro 的 tcp_offset_y
  一致、24 mm 方块的中心在工作面上方 12 mm、夹它需要 26 mm 开口
- perception/README 与根 README 里"相机未到货"改成 Gemini 335L 已到货

验证：tools/run_checks.py 15 项全绿。

File: dummy_vc_ws/src/dummy2_urdf/urdf/dummy2_urdf.xacro (robot description, xacro)
@@ -14,6 +14,11 @@
 <!-- 手指伸出的方向：URDF 里手爪挂在 link7 的 +y 方向 -->
 <xacro:property name="hand_axis" value="y"/>
-<!-- link7 -> 两指夹持中心(指尖前端中点)，沿 hand_axis 的距离。实测 -->
-<xacro:property name="tcp_offset_y" value="0.06"/>
+<!-- link7 -> 两指夹持中心(指尖前端中点)，沿 hand_axis 的距离。
+     实测：2026-10-16 尺量，约 15 mm。
+     注意它比 hand 关节的 0.052312 还小，所以 gripper_tcp 落在 hand 坐标系
+     原点的**后方**（y = 0.015 - 0.052312 = -0.037312，即比 hand 原点更靠近
+     link7）—— 实物手爪的两指是贴着腕部夹的。URDF 里那套手指几何来自原作者
+     模型、与实物不符（docs/04 A1），两者不能互相印证。 -->
+<xacro:property name="tcp_offset_y" value="0.015"/>
 <!-- 相机的安装参数（外置支架，eye-to-hand）定义在文件末尾的相机段落里，
      因为那里有较长的说明。用 grep 搜 camera_offset 可以找到。 -->

Commit message: fix: 相机挂载姿态换成实测位置，并把光学系的归属让给驱动
两件事，都是为了能在真机上空跑 vision_node：

1. camera_link 的挂载从占位值 (0.30, 0, 0.60) / rpy(180,0,0) 换成用户口头给的
   (-0.23, 0.30, 0.15) / rpy(0, 90°, 0)。原来的 rpy 是错的：camera_link 的 +x
   才是镜头方向（光学系的 z 落在它上面），要让镜头朝下必须把 +x 转到 -z，
   也就是绕 y 轴 +90°。按老值算出来光轴指向 base_link 的 +x（水平），
   反投影出来的东西全是斜的，而且不报错。

2. camera_color_optical_frame 从 URDF 里删掉。orbbec_camera 驱动自己发布
   camera_link -> camera_color_frame -> camera_color_optical_frame，URDF 再
   定义一份同名坐标系，那个 frame 就有两个父节点，TF 树两条边；查出来的变换
   不可信，而且失败方式是静默的（数字不对，不报错）。URDF 只保留挂载关节
   base_link -> camera_link，加上一个**不同名**的 usb_camera_optical_frame
   给裸 USB 相机兜底（fingerprint_camera.py 用它，那条路没有驱动发 TF）。

   连带改了三处描述：tools/check_urdf.py 的必需坐标系列表、geometry.py 的
   轴向约定注释、perception README 的坐标轴约定与"还差什么"第 2 条。

验证：run_checks ALL 15 CHECKS PASSED；selftest_vision_geometry 现在报
"占位相机：位置 (-0.23, 0.3, 0.15)，光轴在 base_link 里指向 (0.000, 0.000,
-1.000)"，之前那条"并没有朝下"的 note 消失了。检查仍是 2 条 note（单目偏差
7.1 mm、45° 摆放要 33.9 mm 开口）。挂载位置仍然是估算值，手眼标定后要替换。

File: dummy_vc_ws/src/dummy2_urdf/urdf/dummy2_urdf.xacro (robot description, xacro)
@@ -358,5 +358,9 @@
      坐标链（注意：XML 注释里不能出现连续两个连字符，所以这里用箭头文字替代）
        link7_v1_1  ->  tool0  ->  gripper_tcp
-                           ->  camera_link  ->  camera_color_optical_frame
+                           ->  camera_link  ->  usb_camera_optical_frame
+      相机链其实挂在 base_link 下，不在末端：
+        base_link -> camera_link -> usb_camera_optical_frame（本文件发布，USB 兜底）
+                                -> camera_color_frame -> camera_color_optical_frame
+                                   （后两个由 orbbec_camera 驱动发布）
      ========================================================================== -->
 <!-- tool0：末端法兰坐标，与手爪根部重合，便于标定和参考项目对齐 -->
@@ -388,12 +392,19 @@
          方案 B：给下面这个关节加条件，标定后不再展开
        首期用方案 A，简单直接。 -->
-<xacro:property name="camera_offset_x" value="0.30"/>
-<xacro:property name="camera_offset_y" value="0.0"/>
-<xacro:property name="camera_offset_z" value="0.60"/>
-<!-- 相机安装姿态（度）。外置俯视支架通常是「朝下看」，
-     对应绕 x 轴 -90°；然后再绕 z 轴转一个安装偏航角。
-     这些都是标定前的估计值，手眼标定会给出准确结果。 -->
-<xacro:property name="camera_mount_roll_deg" value="180"/>
-<xacro:property name="camera_mount_pitch_deg" value="0"/>
+<xacro:property name="camera_offset_x" value="-0.23"/>
+<xacro:property name="camera_offset_y" value="0.30"/>
+<xacro:property name="camera_offset_z" value="0.15"/>
+<!-- 相机安装姿态（度）。
+     这三条是 2026-10-16 用户口头给的位置（-x 23 cm、+y 30 cm、高 15 cm），
+     **不是标定结果**，手眼标定会给出准确值。
+     rpy 这里为什么是 pitch=+90° 而不是"绕 x 轴 -90°"：
+     相机本体系 camera_link 的 **+x 是镜头方向**（REP-103 下 x 前），而
+     orbbec_camera 驱动把光学系定义成 optical 的 z（前）指向 camera_link 的 +x。
+     所以要让镜头朝下（optical z = base_link -z），必须把 camera_link 的 +x
+     转到 -z 上，也就是绕 y 轴 +90°。写成绕 x 转 -90° 的话镜头会保持水平朝
+     +x —— 那个值反投影出来的结果全是斜的，而且不会报错。
+     安装偏航角（图像落在哪个方向上）标定前不关心，先取 0。 -->
+<xacro:property name="camera_mount_roll_deg" value="0"/>
+<xacro:property name="camera_mount_pitch_deg" value="90"/>
 <xacro:property name="camera_mount_yaw_deg" value="0"/>
 <link name="camera_link"/>
@@ -404,18 +415,22 @@
   <child link="camera_link"/>
 </joint>
-<!-- camera_color_optical_frame：光学坐标系（z 前、x 右、y 下）。
+<!-- usb_camera_optical_frame：USB 兜底相机的光学坐标系（z 前、x 右、y 下）。
      注意 optical frame 的轴向约定与 REP-103 不同，这是写视觉变换时最容易
      翻车的地方：图像的 x 对应光学系的 x（右），图像的 y 对应光学系的 y（下），
      深度对应光学系的 z（前，正值朝景物）。
-     RealSense 的 realsense2_camera 节点会自己发布 camera_link 到
-     camera_color_optical_frame，所以接了真实驱动后这里会被覆盖；
-     保留它是为了没有相机时 RViz 里也能看到坐标系。
+     camera_color_optical_frame 不在这里定义 —— 它由 orbbec_camera 驱动自己发布
+     （camera_link -> camera_color_frame -> camera_color_optical_frame）。
+     以前这里也定义过一份同名的，结果是那个 frame 同时挂在 xacro 的
+     camera_link 与驱动的 camera_color_frame 两个父节点下，TF 树出现两条边；
+     查出来的变换不可信，而且不报错，只是数字不对。两个名字分开之后，
+     接 Gemini 用驱动的 camera_color_optical_frame，跑裸 USB 相机用本文件的
+     usb_camera_optical_frame，互不干扰。
      rpy="-1.5707963 0 -1.5707963" 是 REP-103 -> 光学系的标准变换：
      绕 x 转 -90° 把 z 从朝上掰到朝前，再绕 z 转 -90° 对齐 x/y。 -->
-<link name="camera_color_optical_frame"/>
-<joint name="camera_optical_joint" type="fixed">
+<link name="usb_camera_optical_frame"/>
+<joint name="usb_camera_optical_joint" type="fixed">
   <origin xyz="0 0 0" rpy="-1.5707963 0 -1.5707963"/>
   <parent link="camera_link"/>
-  <child link="camera_color_optical_frame"/>
+  <child link="usb_camera_optical_frame"/>
 </joint>
 </robot>

Commit message: fix: 相机是斜下 30° 不是垂直向下 —— 挂载姿态和那条"不朝下"的检查
用户补充：相机与水平面约成 30° 斜向下，方块在 base_link 的 +y 31 cm 处。
原来那两个数（pitch=90°、门限轴 -0.7）都是按"垂直俯视"写的，两个都错了。

1. xacro 的 camera_mount_pitch_deg 90 → 30。camera_link 的 +x 是镜头方向，
   绕 y 转 pitch 才是把镜头压低的那一次转动：pitch=90° 垂直朝下，
   pitch=30° 就是斜下 30°，光轴 (0.866, 0, -0.500)，落地点 (+0.03, +0.30, 0)
   —— 离方块 ((0, +0.31, 0)) 只有几厘米，所以方块该出现在画面中心附近。

2. vision_node 那个"光轴不是朝下"的警告门限从 axis[2] > -0.7 改成 > -0.3。
   斜下 30° 的竖直分量是 -0.50，老门限会把它当成装歪了、每帧刷假警报。
   改成"只要明显朝下（约 17° 以上）就放过"，真正要挡的是"几乎水平"
   （rpy 写成 roll=180 时 axis[2] = 0，那种相机照不到工作面）。

3. selftest 第 7 组从"只提示不判红"升级成真检查：光轴竖直分量必须 < -0.3，
   否则判红并说明原因。同时把实测的俯角打进 note：斜视在倾斜方向上误差被
   1/sin 放大（30° 时约 2 倍），画面远端更差，所以方块要放画面中部。

实算（1280×720、fx 614、斜下 30°、相机在 (-0.23, 0.30, 0.15)）：
方块中心投到像素 (619, 376)，画面中心是 (640, 360)，基本正中；方块那个距离
0.268 m 上 1 像素 ≈ 0.44 mm；画面上方有一块在地平线以上（打无穷远，会被丢掉）。

验证：run_checks ALL 15 CHECKS PASSED；selftest_vision_geometry 输出
"光轴在 base_link 里指向 (0.866, 0.000, -0.500)（低于水平面 30.0°）"，
3 条 note（斜视放大 2 倍、单目 7.1 mm、45° 摆放要 33.9 mm 开口）。

File: dummy_vc_ws/src/dummy2_urdf/urdf/dummy2_urdf.xacro (robot description, xacro)
@@ -398,13 +398,21 @@
      这三条是 2026-10-16 用户口头给的位置（-x 23 cm、+y 30 cm、高 15 cm），
      **不是标定结果**，手眼标定会给出准确值。
-     rpy 这里为什么是 pitch=+90° 而不是"绕 x 轴 -90°"：
+     相机是**斜向下 30°（相对水平）**，不是垂直向下 —— 倾斜方向朝 +x，
+     光轴在 base_link 里是 (0.866, 0, -0.500)，落到地面（z=0）上的点是
+     (-0.23 + 0.15/tan30°, 0.30) ≈ (+0.03, +0.30)，离用户说的方块位置
+     （+y 31 cm、x≈0）只有几厘米，所以方块应该出现在画面中心附近。
+     rpy 这里为什么是 pitch=+30°：
      相机本体系 camera_link 的 **+x 是镜头方向**（REP-103 下 x 前），而
      orbbec_camera 驱动把光学系定义成 optical 的 z（前）指向 camera_link 的 +x。
-     所以要让镜头朝下（optical z = base_link -z），必须把 camera_link 的 +x
-     转到 -z 上，也就是绕 y 轴 +90°。写成绕 x 转 -90° 的话镜头会保持水平朝
-     +x —— 那个值反投影出来的结果全是斜的，而且不会报错。
-     安装偏航角（图像落在哪个方向上）标定前不关心，先取 0。 -->
+     绕 y 轴转 pitch 角，+x 变成 (cos pitch, 0, -sin pitch)：
+       pitch=90° → (0, 0, -1)  垂直朝下
+       pitch=30° → (0.866, 0, -0.5)  朝 +x 斜下 30°  ← 现在用这个
+     写成绕 x 轴转 roll 的话镜头只在 yz 平面里动，方向完全不同；写成
+     roll=180 则镜头水平朝 +x —— 那个值反投影出来的结果全是斜的，而且
+     不会报错。
+     yaw=0：倾斜方向就是 +x。如果实机上画面中心不在方块上，改的是 pitch
+     和 yaw 两个数（pitch 管压低多少、yaw 管朝哪个方位压），不是只改 yaw。 -->
 <xacro:property name="camera_mount_roll_deg" value="0"/>
-<xacro:property name="camera_mount_pitch_deg" value="90"/>
+<xacro:property name="camera_mount_pitch_deg" value="30"/>
 <xacro:property name="camera_mount_yaw_deg" value="0"/>
 <link name="camera_link"/>
