Commit message: fix: 手掌盒子的背面和 link6 的正面重合，起始位姿被判成自碰撞
真机日志：Found a contact between 'link6_v3_1' and 'dummy_hand_v1_1' /
Start state appears to be in collision / Unable to find a valid state nearby。

不是盒子太大：joint6 的 origin 就在 link6 网格的最大 y（0.1185），而 joint6 的轴
是 (0,-1,0)，所以 link7（和它上面的手掌）只会在关节平面之外。我把手掌盒子的
背面正好放在 link7 的 y=0 上 —— 与 link6 的正面同一个平面，FCL 把面接触算成
碰撞，于是起始状态永远不可规划。

往 +y 挪 1 mm（新 property gripper_seam_gap_m）让两个面分开；手指、TCP、
抓取点都不在那一侧，数值不受影响。

顺带在 tools/check_urdf.py 里加了一条离线判据：gripper_seam_gap_m >= 1 mm
且手掌盒子的 origin 真的用上了它 —— 这类错误只有在装了 FCL 的机器上才暴露，
等真机上再撞一次太贵。

File: dummy_vc_ws/src/dummy2_urdf/urdf/dummy2_urdf.xacro (robot description, xacro)
@@ -40,4 +40,10 @@
 <!-- 半行程 = 一指从全闭到全开走多远 -->
 <xacro:property name="gripper_finger_travel_m" value="${gripper_open_gap_m/2}"/>
+<!-- 手掌盒子的背面和 link6 的正面正好在同一个平面上（joint6 的 origin y
+     就是 link6 网格的最大 y = 0.1185），FCL 把"面接触"也算碰撞，于是起始
+     状态永远被判成自碰撞：Found a contact between 'link6_v3_1' and
+     'dummy_hand_v1_1' / Start state appears to be in collision。往 +y 挪
+     1 mm 让两个面分开；手指、TCP、抓取点都不受影响（手指在更外面）。 -->
+<xacro:property name="gripper_seam_gap_m" value="0.001"/>
 <!-- link7 端面 -> 两指夹持中心（gripper_tcp 就放在这里） -->
 <xacro:property name="tcp_offset_y" value="${gripper_wrist_to_tip_m - gripper_tip_to_centre_m}"/>
@@ -204,7 +210,8 @@
   <!-- 手掌/舵机本体：用实测尺寸的盒体，不用原作者网格（见文件上方 A1 注释）。
        本体从腕部往指尖方向占 80 mm，所以盒心在 hand 坐标系
-       y = 80/2 - 52.312 = -12.3 mm。 -->
-  <visual>
-    <origin xyz="0 ${gripper_body_y_m/2 - 0.052312} 0" rpy="0 0 0"/>
+       y = 80/2 - 52.312 + 1 = -11.3 mm —— 那个 +1 mm 是 gripper_seam_gap_m，
+       把背面和 link6 的正面（同一平面）分开，否则面接触被判成自碰撞。 -->
+  <visual>
+    <origin xyz="0 ${gripper_body_y_m/2 - 0.052312 + gripper_seam_gap_m} 0" rpy="0 0 0"/>
     <geometry>
       <box size="${gripper_body_x_m} ${gripper_body_y_m} ${gripper_body_z_m}"/>
@@ -213,5 +220,5 @@
   </visual>
   <collision>
-    <origin xyz="0 ${gripper_body_y_m/2 - 0.052312} 0" rpy="0 0 0"/>
+    <origin xyz="0 ${gripper_body_y_m/2 - 0.052312 + gripper_seam_gap_m} 0" rpy="0 0 0"/>
     <geometry>
       <box size="${gripper_body_x_m} ${gripper_body_y_m} ${gripper_body_z_m}"/>
